Commit message: edits and thruster definition

File: auv_description/urdf/auv.urdf.xacro (robot description, xacro)
@@ -1,17 +1,17 @@
 <?xml version="1.0"?>
 <robot xmlns:xacro="http://www.ros.org/wiki/xacro" name="2dof_robot">
-  <xacro:arg name="prefix" default="" />
+  <xacro:arg name="prefix" default="auv"/>
   <!-- Import RRBot macro -->
-  <xacro:include filename="$(find auv_description)/urdf/auv_description.urdf.xacro" />
+  <xacro:include filename="$(find auv_description)/urdf/auv_description.urdf.xacro"/>
   <!-- Import Rviz colors -->
-  <xacro:include filename="$(find auv_description)/urdf/auv.materials.xacro" />
+  <xacro:include filename="$(find auv_description)/urdf/auv.materials.xacro"/>
   <!-- Import RRBot ros2_control description -->
-  <xacro:include filename="$(find auv_description)/urdf/auv.ros2_control.xacro" />
+  <xacro:include filename="$(find auv_description)/urdf/auv.ros2_control.xacro"/>
   <!-- Used for fixing robot -->
   <!-- <link name="world" /> -->
   <xacro:auv_bot parent="world"
     prefix="$(arg prefix)">
-    <origin xyz="0 0 0" rpy="0 0 0" />
+    <origin xyz="0 0 0" rpy="0 0 0"/>
   </xacro:auv_bot>
-  <xacro:auv_ros2_control name="auv" prefix="$(arg prefix)" />
+  <xacro:auv_ros2_control name="auv_hw_interface" prefix="$(arg prefix)"/>
 </robot>

File: auv_description/urdf/auv_description.urdf.xacro (robot description, xacro)
@@ -2,60 +2,70 @@
 <robot xmlns:xacro="http://www.ros.org/wiki/xacro">
   <xacro:macro name="auv_bot" params="parent prefix *origin">
-    <!-- Constants for robot dimensions -->
-    <xacro:property name="mass" value="1" /> <!-- arbitrary value for mass -->
-    <xacro:property name="width" value="0.1" /> <!-- Square dimensions (widthxwidth) of beams -->
-    <xacro:property name="height1" value="2" /> <!-- Link 1 -->
-    <xacro:property name="height2" value="1" /> <!-- Link 2 -->
-    <xacro:property name="height3" value="1" /> <!-- Link 3 -->
-    <xacro:property name="axel_offset" value="0.05" /> <!-- Space btw top of beam and the each joint -->
     <!-- Base Link -->
-    <link name="${prefix}base_link">
+    <link name="${prefix}/base_link">
       <visual>
-        <origin xyz="0 0 0" rpy="0 0 0" />
+        <origin xyz="0 0 0" rpy="0 0 0"/>
         <geometry>
-          <box size="0.1 0.1 0.1" />
+          <box size="0.1 0.1 0.1"/>
         </geometry>
-        <material name="orange" />
+        <material name="orange"/>
       </visual>
     </link>
     <!-- Middle Link -->
-    <link name="${prefix}link1">
+    <link name="${prefix}/link1">
       <collision>
-        <origin xyz="0 0 ${height2/2 - axel_offset}" rpy="0 0 0" />
+        <origin xyz="0 0 0" rpy="0 0 0"/>
         <geometry>
-          <box size="${width} ${width} ${height2}" />
+          <box size="0 0 0"/>
         </geometry>
       </collision>
       <visual>
-        <origin xyz="0 0 ${height2/2 - axel_offset}" rpy="0 0 0" />
+        <origin xyz="0 0 0" rpy="0 0 0"/>
         <geometry>
-          <box size="${width} ${width} ${height2}" />
+          <box size="0 0 0"/>
         </geometry>
-        <material name="yellow" />
+        <material name="yellow"/>
       </visual>
     </link>
     <!-- Top Link -->
-    <link name="${prefix}link2">
+    <link name="${prefix}/link2">
       <visual>
-        <origin xyz="0 0 ${height3/2 - axel_offset}" rpy="0 0 0" />
+        <origin xyz="0 0 0" rpy="0 0 0"/>
         <geometry>
-          <box size="${width} ${width} ${height3}" />
+          <box size="0 0 0"/>
         </geometry>
-        <material name="orange" />
+        <material name="orange"/>
       </visual>
     </link>
-    <joint name="${prefix}joint1" type="continuous">
-      <parent link="${prefix}base_link" />
-      <child link="${prefix}link1" />
-      <origin xyz="0 ${width} ${height1 - axel_offset}" rpy="0 0 0" />
-      <axis xyz="0 1 0" />
-      <limit effort="100" velocity="1.0" />
+    <joint name="${prefix}/joint1" type="continuous">
+      <parent link="${prefix}/base_link"/>
+      <child link="${prefix}/link1"/>
+      <origin xyz="0 0 0" rpy="0 0 0"/>
+      <axis xyz="0 1 0"/>
+      <limit effort="100" velocity="1.0"/>
     </joint>
-    <joint name="${prefix}joint2" type="continuous">
-      <parent link="${prefix}link1" />
-      <child link="${prefix}link2" />
-      <origin xyz="0 ${width} ${height2 - axel_offset*2}" rpy="0 0 0" />
-      <axis xyz="0 1 0" />
-      <limit effort="100" velocity="1.0" />
+    <joint name="${prefix}/joint2" type="continuous">
+      <parent link="${prefix}/link1"/>
+      <child link="${prefix}/link2"/>
+      <origin xyz="0 0 0" rpy="0 0 0"/>
+      <axis xyz="0 1 0"/>
+      <limit effort="100" velocity="1.0"/>
+    </joint>
+    <!-- Thrusters -->
+    <link name="${prefix}/thruster3"/>
+    <link name="${prefix}/thruster4"/>
+    <joint name="${prefix}/thruster3_joint" type="continuous">
+      <parent link="${prefix}/base_link"/>
+      <child link="${prefix}/thruster3"/>
+      <origin xyz="-0.35 0.35 0" rpy="0 0 0.785398"/>
+      <axis xyz="1 0 0"/>
+      <limit effort="100" velocity="1.0"/>
+    </joint>
+    <joint name="${prefix}/thruster4_joint" type="continuous">
+      <parent link="${prefix}/base_link"/>
+      <child link="${prefix}/thruster4"/>
+      <origin xyz="-0.35 -0.35 0" rpy="0 0 -0.785398"/>
+      <axis xyz="1 0 0"/>
+      <limit effort="100" velocity="1.0"/>
     </joint>
   </xacro:macro>
