Commit message: using udrf file now

File: auv_description/urdf/auv.ros2_control.xacro (robot description, xacro)
@@ -1,12 +1,17 @@
 <?xml version="1.0"?>
 <robot xmlns:xacro="http://www.ros.org/wiki/xacro">
-  <xacro:macro name="rrbot_ros2_control" params="name prefix">
+  <xacro:macro name="auv_ros2_control" params="name prefix">
     <ros2_control name="${name}" type="system">
+      <!-- hardware interface mock/stonefish/real_thruster -->
       <hardware>
-        <plugin>ros2_control_demo_example_1/RRBotSystemPositionOnlyHardware</plugin>
-        <param name="example_param_hw_start_duration_sec">0</param>
-        <param name="example_param_hw_stop_duration_sec">3.0</param>
-        <param name="example_param_hw_slowdown">100</param>
+        <plugin>mock_components/GenericSystem</plugin>
+        <param name="calculate_dynamics">true</param>
       </hardware>
+      <!-- <hardware>
+        <plugin>StonefishHardwareInterface/ThrusterCommand</plugin>
+      </hardware> -->
+      <!-- <thruster>
+      <param name="maxSetpoint">300</param>
+      </thruster> -->
       <joint name="${prefix}joint1">
         <command_interface name="position">
@@ -14,5 +19,5 @@
           <param name="max">1</param>
         </command_interface>
-        <state_interface name="position"/>
+        <state_interface name="position" />
       </joint>
       <joint name="${prefix}joint2">
@@ -21,5 +26,5 @@
           <param name="max">1</param>
         </command_interface>
-        <state_interface name="position"/>
+        <state_interface name="position" />
       </joint>
     </ros2_control>

File: auv_description/urdf/auv.urdf.xacro (robot description, xacro)
@@ -1,21 +1,17 @@
 <?xml version="1.0"?>
-<!-- Revolute-Revolute Manipulator -->
-<!--
-Copied and modified from ROS1 example -
-https://github.com/ros-simulation/gazebo_ros_demos/blob/kinetic-devel/rrbot_description/urdf/rrbot.xacro
--->
 <robot xmlns:xacro="http://www.ros.org/wiki/xacro" name="2dof_robot">
   <xacro:arg name="prefix" default="" />
   <!-- Import RRBot macro -->
-  <xacro:include filename="$(find roscontrol_test)/urdf/rrbot_description.urdf.xacro" />
-    <!-- Import Rviz colors -->
-  <xacro:include filename="$(find roscontrol_test)/urdf/rrbot.materials.xacro" />
+  <xacro:include filename="$(find auv_description)/urdf/auv_description.urdf.xacro" />
+  <!-- Import Rviz colors -->
+  <xacro:include filename="$(find auv_description)/urdf/auv.materials.xacro" />
   <!-- Import RRBot ros2_control description -->
-  <!-- <xacro:include filename="$(find ros2_control_demo_example_1)/ros2_control/rrbot.ros2_control.xacro" /> -->
+  <xacro:include filename="$(find auv_description)/urdf/auv.ros2_control.xacro" />
   <!-- Used for fixing robot -->
-  <!-- <link name="world"/> -->
-  <xacro:rrbot parent="world" prefix="$(arg prefix)">
+  <!-- <link name="world" /> -->
+  <xacro:auv_bot parent="world"
+    prefix="$(arg prefix)">
     <origin xyz="0 0 0" rpy="0 0 0" />
-  </xacro:rrbot>
-  <!-- <xacro:rrbot_ros2_control name="RRBot" prefix="$(arg prefix)" /> -->
+  </xacro:auv_bot>
+  <xacro:auv_ros2_control name="auv" prefix="$(arg prefix)" />
 </robot>

Commit message: testing stonefish hardware interface

File: auv_description/urdf/auv.ros2_control.xacro (robot description, xacro)
@@ -4,11 +4,11 @@
     <ros2_control name="${name}" type="system">
       <!-- hardware interface mock/stonefish/real_thruster -->
-      <hardware>
+      <!-- <hardware>
         <plugin>mock_components/GenericSystem</plugin>
         <param name="calculate_dynamics">true</param>
+      </hardware> -->
+      <hardware>
+        <plugin>stonefish_hw_interface/ThrusterGroupHWInterface</plugin>
       </hardware>
-      <!-- <hardware>
-        <plugin>StonefishHardwareInterface/ThrusterCommand</plugin>
-      </hardware> -->
       <!-- <thruster>
       <param name="maxSetpoint">300</param>

File: auv_description/urdf/auv_description.urdf.xacro (robot description, xacro)
@@ -1,5 +1,5 @@
 <?xml version="1.0"?>
 <robot xmlns:xacro="http://www.ros.org/wiki/xacro">
-  <xacro:macro name="rrbot" params="parent prefix *origin">
+  <xacro:macro name="auv_bot" params="parent prefix *origin">
     <!-- Constants for robot dimensions -->
     <xacro:property name="mass" value="1" /> <!-- arbitrary value for mass -->

Commit message: urdf hardware thruster definition

File: auv_description/urdf/auv.ros2_control.xacro (robot description, xacro)
@@ -10,21 +10,21 @@
       <hardware>
         <plugin>stonefish_hw_interface/ThrusterGroupHWInterface</plugin>
+        <param name="thruster_group_write_topic">auv/sf_controller/thruster_setpoints_sim</param>
+        <param name="thruster_group_read_topic">auv/sf_controller/thruster_state</param>
       </hardware>
       <!-- <thruster>
       <param name="maxSetpoint">300</param>
       </thruster> -->
-      <joint name="${prefix}joint1">
-        <command_interface name="position">
-          <param name="min">-1</param>
-          <param name="max">1</param>
+      <joint name="${prefix}/thruster3_joint">
+        <command_interface name="velocity">
+          <param name="max_setpoint">100</param>
         </command_interface>
-        <state_interface name="position" />
+        <state_interface name="velocity"/>
       </joint>
-      <joint name="${prefix}joint2">
-        <command_interface name="position">
-          <param name="min">-1</param>
-          <param name="max">1</param>
+      <joint name="${prefix}/thruster4_joint">
+        <command_interface name="velocity">
+          <param name="max_setpoint">100</param>
         </command_interface>
-        <state_interface name="position" />
+        <state_interface name="velocity"/>
       </joint>
     </ros2_control>

Commit message: added bow and stern thrusters

File: auv_description/urdf/auv.ros2_control.xacro (robot description, xacro)
@@ -13,7 +13,4 @@
         <param name="thruster_group_read_topic">auv/sf_controller/thruster_state</param>
       </hardware>
-      <!-- <thruster>
-      <param name="maxSetpoint">300</param>
-      </thruster> -->
       <joint name="${prefix}/thruster3_joint">
         <command_interface name="velocity">
@@ -28,4 +25,16 @@
         <state_interface name="velocity"/>
       </joint>
+      <joint name="${prefix}/thruster5_joint">
+        <command_interface name="velocity">
+          <param name="max_setpoint">100</param>
+        </command_interface>
+        <state_interface name="velocity"/>
+      </joint>
+      <joint name="${prefix}/thruster6_joint">
+        <command_interface name="velocity">
+          <param name="max_setpoint">100</param>
+        </command_interface>
+        <state_interface name="velocity"/>
+      </joint>
     </ros2_control>
   </xacro:macro>

File: auv_description/urdf/auv_description.urdf.xacro (robot description, xacro)
@@ -55,4 +55,6 @@
     <link name="${prefix}/thruster3"/>
     <link name="${prefix}/thruster4"/>
+    <link name="${prefix}/thruster5"/>
+    <link name="${prefix}/thruster6"/>
     <joint name="${prefix}/thruster3_joint" type="continuous">
       <parent link="${prefix}/base_link"/>
@@ -69,4 +71,18 @@
       <limit effort="100" velocity="1.0"/>
     </joint>
+    <joint name="${prefix}/thruster5_joint" type="continuous">
+      <parent link="${prefix}/base_link"/>
+      <child link="${prefix}/thruster5"/>
+      <origin xyz="0.60 0 0" rpy="0 0 0"/>
+      <axis xyz="1 0 0"/>
+      <limit effort="100" velocity="1.0"/>
+    </joint>
+    <joint name="${prefix}/thruster6_joint" type="continuous">
+      <parent link="${prefix}/base_link"/>
+      <child link="${prefix}/thruster6"/>
+      <origin xyz="-0.60 0.0 0" rpy="0 0 0"/>
+      <axis xyz="1 0 0"/>
+      <limit effort="100" velocity="1.0"/>
+    </joint>
   </xacro:macro>
 </robot>
